File: FLAMENCOFLOCK/FLAMENCOFLOCK.sch (KiCad schematic (older format))
At the start: 8 parts, among them J1 MINIDIN6, J2 MINIDIN6, P2 ANTENNA, Q1 MOSFET_N

Commit message: finished FLAMENCOFLOCK
Parts:
- removed R1: DNP, symbol R
- removed R3, R4: 0, symbol R
Connections:
- wire segments 28 -> 24
Other:
- note removed: "Cut trace to install\nresistor on R3 or R4."
- moved on the sheet: P2, Q1, R2
Changed lines of the file:
@@
-EESchema Schematic File Version 2  date Mon 28 Jul 2014 11:41:41 AM MDT
+EESchema Schematic File Version 2  date Mon 28 Jul 2014 08:57:02 PM MDT
 LIBS:power
 LIBS:device
@@
 Sheet 1 1
 Title "FLAMENCOFLOCK"
-Date "28 jul 2014"
+Date "29 jul 2014"
 Rev ""
 Comp "Copyright 2014 Michael Ossmann"
@@
 L MOSFET_N Q1
 U 1 1 5370319E
-P 4750 2250
-F 0 "Q1" H 4760 2420 60  0000 R CNN
-F 1 "MOSFET_N" V 4950 2450 60  0000 R CNN
-F 4 "NXP" H 4750 2250 60  0001 C CNN "Manufacturer"
-F 5 "BSS83,215" H 4750 2250 60  0001 C CNN "Part Number"
-F 6 "MOSFET N-CH 10V 50MA SOT-143B" H 4750 2250 60  0001 C CNN "Description"
-	1    4750 2250
+P 4250 2250
+F 0 "Q1" H 4260 2420 60  0000 R CNN
+F 1 "MOSFET_N" V 4450 2450 60  0000 R CNN
+F 4 "NXP" H 4250 2250 60  0001 C CNN "Manufacturer"
+F 5 "BSS83,215" H 4250 2250 60  0001 C CNN "Part Number"
+F 6 "MOSFET N-CH 10V 50MA SOT-143B" H 4250 2250 60  0001 C CNN "Description"
+	1    4250 2250
 	1    0    0    -1
 $EndComp
 Wire Wire Line
-	4850 1450 4850 2050
+	4350 1450 4350 2050
 Wire Wire Line
-	3750 2250 4550 2250
+	2400 2250 4050 2250
 $Comp
 L R R2
 U 1 1 53703213
-P 4500 2550
-F 0 "R2" V 4580 2550 50  0000 C CNN
-F 1 "10k" V 4500 2550 50  0000 C CNN
-	1    4500 2550
+P 4000 2550
+F 0 "R2" V 4080 2550 50  0000 C CNN
+F 1 "10k" V 4000 2550 50  0000 C CNN
+	1    4000 2550
 	0    -1   -1   0
 $EndComp
-Connection ~ 4150 2250
+Connection ~ 3650 2250
 $Comp
-L R R1
-U 1 1 5370DAFA
-P 5200 1950
-F 0 "R1" V 5280 1950 50  0000 C CNN
-F 1 "DNP" V 5200 1950 50  0000 C CNN
-F 4 "DNP" V 5100 1950 60  0000 C CNN "Note"
-	1    5200 1950
+L GND #PWR01
+U 1 1 5370DB21
+P 4350 2950
+F 0 "#PWR01" H 4350 2950 30  0001 C CNN
+F 1 "GND" H 4350 2880 30  0001 C CNN
+	1    4350 2950
+	1    0    0    -1
+$EndComp
+Wire Wire Line
+	3650 2250 3650 2550
+Wire Wire Line
+	3650 2550 3750 2550
+Wire Wire Line
+	4250 2550 4350 2550
+Connection ~ 4350 2550
+$Comp
+L CONN_2 P2
+U 1 1 53B03152
+P 4450 1100
+F 0 "P2" V 4400 1100 40  0000 C CNN
+F 1 "ANTENNA" V 4500 1100 40  0000 C CNN
+	1    4450 1100
 	0    -1   -1   0
 $EndComp
 $Comp
-L R R3
-U 1 1 5370DB07
-P 4850 3250
-F 0 "R3" V 4930 3250 50  0000 C CNN
-F 1 "0" V 4850 3250 50  0000 C CNN
-F 4 "DNP" V 4750 3250 60  0000 C CNN "Note"
-	1    4850 3250
-	-1   0    0    1
-$EndComp
-$Comp
-L GND #PWR01
-U 1 1 5370DB21
-P 4850 3600
-F 0 "#PWR01" H 4850 3600 30  0001 C CNN
-F 1 "GND" H 4850 3530 30  0001 C CNN
-	1    4850 3600
-	1    0    0    -1
-$EndComp
-$Comp
 L GND #PWR02
-U 1 1 5370DB27
-P 5550 1950
-F 0 "#PWR02" H 5550 1950 30  0001 C CNN
-F 1 "GND" H 5550 1880 30  0001 C CNN
-	1    5550 1950
-	0    -1   -1   0
-$EndComp
-Wire Wire Line
-	5550 1950 5450 1950
-Wire Wire Line
-	4950 1950 4850 1950
-Connection ~ 4850 1950
-Wire Wire Line
-	4850 2450 4850 3000
-Wire Wire Line
-	4850 3600 4850 3500
-Wire Wire Line
-	4150 2250 4150 2550
-Wire Wire Line
-	4150 2550 4250 2550
-Wire Wire Line
-	4750 2550 4850 2550
-Connection ~ 4850 2550
-$Comp
-L CONN_2 P2
-U 1 1 53B03152
-P 4950 1100
-F 0 "P2" V 4900 1100 40  0000 C CNN
-F 1 "ANTENNA" V 5000 1100 40  0000 C CNN
-	1    4950 1100
-	0    -1   -1   0
-$EndComp
-$Comp
-L GND #PWR03
 U 1 1 53B0316B
-P 5050 1550
-F 0 "#PWR03" H 5050 1550 30  0001 C CNN
-F 1 "GND" H 5050 1480 30  0001 C CNN
-	1    5050 1550
+P 4550 1550
+F 0 "#PWR02" H 4550 1550 30  0001 C CNN
+F 1 "GND" H 4550 1480 30  0001 C CNN
+	1    4550 1550
 	1    0    0    -1
 $EndComp
 Wire Wire Line
-	5050 1450 5050 1550
+	4550 1450 4550 1550
 $Comp
-L GND #PWR04
+L GND #PWR03
 U 1 1 53B031B0
-P 3850 3150
-F 0 "#PWR04" H 3850 3150 30  0001 C CNN
-F 1 "GND" H 3850 3080 30  0001 C CNN
-	1    3850 3150
+P 3300 2600
+F 0 "#PWR03" H 3300 2600 30  0001 C CNN
+F 1 "GND" H 3300 2530 30  0001 C CNN
+	1    3300 2600
 	1    0    0    -1
 $EndComp
-Wire Wire Line
-	3750 2450 3850 2450
-Wire Wire Line
-	3850 2450 3850 2550
-$Comp
-L R R4
-U 1 1 53B032AD
-P 3850 2800
-F 0 "R4" V 3930 2800 50  0000 C CNN
-F 1 "0" V 3850 2800 50  0000 C CNN
-F 4 "DNP" V 3750 2800 60  0000 C CNN "Note"
-	1    3850 2800
-	-1   0    0    1
-$EndComp
-Wire Wire Line
-	3850 3050 3850 3150
-Text Label 4850 1800 1    40   ~ 0
+Text Label 4350 1800 1    40   ~ 0
 DRAIN
-Text Label 3800 2250 0    40   ~ 0
+Text Label 3300 2250 0    40   ~ 0
 GATE
-Text Label 4850 2850 1    40   ~ 0
+Text Label 4350 2850 1    40   ~ 0
 SOURCE
-Text Notes 4100 3000 0    40   ~ 0
-Cut trace to install\nresistor on R3 or R4.
-Wire Notes Line
-	3850 2550 4000 2550
-Wire Notes Line
-	4000 2550 4000 3050
-Wire Notes Line
-	4000 3050 3850 3050
-Wire Notes Line
-	4850 3000 5000 3000
-Wire Notes Line
-	5000 3000 5000 3500
-Wire Notes Line
-	5000 3500 4850 3500
-Text Notes 5250 1100 0    40   ~ 0
+Text Notes 4750 1100 0    40   ~ 0
 Connect dipole to pins 1 and 2\nor connect monopole to pin 1.
 $Comp
@@
 Text Label 2550 1950 1    40   ~ 0
 SHIELD
+Connection ~ 2400 2250
+Wire Wire Line
+	3300 2600 3300 2500
+Wire Wire Line
+	3300 2500 2950 2500
+Connection ~ 2950 2500
+Wire Wire Line
+	4350 2450 4350 2950
 $EndSCHEMATC

Commit message: connected BSS83,215 substrate to source (previous workaround was solder blob)
Parts:
- Q1: symbol MOSFET_N -> MOS_N4
Connections:
- net GND: now also Q1.B
Changed lines of the file:
@@
-EESchema Schematic File Version 2  date Mon 28 Jul 2014 08:57:02 PM MDT
+EESchema Schematic File Version 2  date Tue 12 Aug 2014 10:41:50 PM MDT
 LIBS:power
 LIBS:device
@@
 Sheet 1 1
 Title "FLAMENCOFLOCK"
-Date "29 jul 2014"
+Date "13 aug 2014"
 Rev ""
 Comp "Copyright 2014 Michael Ossmann"
@@
 $EndDescr
 $Comp
-L MOSFET_N Q1
+L MOS_N4 Q1
 U 1 1 5370319E
 P 4250 2250
@@
 Text Label 3300 2250 0    40   ~ 0
 GATE
-Text Label 4350 2850 1    40   ~ 0
+Text Label 4350 2900 1    40   ~ 0
 SOURCE
 Text Notes 4750 1100 0    40   ~ 0
@@
 Wire Wire Line
 	4350 2450 4350 2950
+Wire Wire Line
+	4400 2250 4500 2250
+Wire Wire Line
+	4500 2250 4500 2650
+Wire Wire Line
+	4500 2650 4350 2650
+Connection ~ 4350 2650
 $EndSCHEMATC
