File: TANGOFLOCK/TANGOFLOCK.sch (KiCad schematic (older format))
At the start: 7 parts, among them J1 USB-DEVICE-SHIELD, J2 USB-DEVICE-SHIELD, P2 ANTENNA, Q1 MOSFET_N

Commit message: simplified TANGOFLOCK
Parts:
- removed R1: DNP, symbol R
- removed R3: 0, symbol R
Connections:
- net SOURCE is gone; now on net GND: Q1.S, R2.2
Other:
- note removed: "Cut trace to install\nresistor on R3."
Changed lines of the file:
@@
-EESchema Schematic File Version 2  date Mon 28 Jul 2014 06:47:18 PM MDT
+EESchema Schematic File Version 2  date Mon 28 Jul 2014 08:58:28 PM MDT
 LIBS:power
 LIBS:device
@@
 Connection ~ 4150 2250
 $Comp
-L R R1
-U 1 1 5370DAFA
-P 5200 1950
-F 0 "R1" V 5280 1950 50  0000 C CNN
-F 1 "DNP" V 5200 1950 50  0000 C CNN
-F 4 "DNP" V 5100 1950 60  0000 C CNN "Note"
-	1    5200 1950
-	0    -1   -1   0
-$EndComp
-$Comp
-L R R3
-U 1 1 5370DB07
-P 4850 3250
-F 0 "R3" V 4930 3250 50  0000 C CNN
-F 1 "0" V 4850 3250 50  0000 C CNN
-F 4 "DNP" V 4750 3250 60  0000 C CNN "Note"
-	1    4850 3250
-	-1   0    0    1
-$EndComp
-$Comp
 L GND #PWR01
 U 1 1 5370DB21
-P 4850 3600
-F 0 "#PWR01" H 4850 3600 30  0001 C CNN
-F 1 "GND" H 4850 3530 30  0001 C CNN
-	1    4850 3600
+P 4850 3000
+F 0 "#PWR01" H 4850 3000 30  0001 C CNN
+F 1 "GND" H 4850 2930 30  0001 C CNN
+	1    4850 3000
 	1    0    0    -1
 $EndComp
-$Comp
-L GND #PWR02
-U 1 1 5370DB27
-P 5550 1950
-F 0 "#PWR02" H 5550 1950 30  0001 C CNN
-F 1 "GND" H 5550 1880 30  0001 C CNN
-	1    5550 1950
-	0    -1   -1   0
-$EndComp
-Wire Wire Line
-	5550 1950 5450 1950
-Wire Wire Line
-	4950 1950 4850 1950
-Connection ~ 4850 1950
 Wire Wire Line
 	4850 2450 4850 3000
-Wire Wire Line
-	4850 3600 4850 3500
 Wire Wire Line
 	4150 2250 4150 2550
@@
 Text Label 4850 2850 1    40   ~ 0
 SOURCE
-Text Notes 5050 3050 0    40   ~ 0
-Cut trace to install\nresistor on R3.
-Wire Notes Line
-	4850 3000 5000 3000
-Wire Notes Line
-	5000 3000 5000 3500
-Wire Notes Line
-	5000 3500 4850 3500
 Text Notes 5250 1100 0    40   ~ 0
 Connect dipole to pins 1 and 2\nor connect monopole to pin 1.

Commit message: connected BSS83,215 substrate to source (previous workaround was solder blob)
Parts:
- Q1: symbol MOSFET_N -> MOS_N4
Connections:
- net GND: now also Q1.B
Changed lines of the file:
@@
-EESchema Schematic File Version 2  date Mon 28 Jul 2014 08:58:28 PM MDT
+EESchema Schematic File Version 2  date Tue 12 Aug 2014 10:43:27 PM MDT
 LIBS:power
 LIBS:device
@@
 Sheet 1 1
 Title "TANGOFLOCK"
-Date "29 jul 2014"
+Date "13 aug 2014"
 Rev ""
 Comp "Copyright 2014 Michael Ossmann"
@@
 $EndDescr
 $Comp
-L MOSFET_N Q1
+L MOS_N4 Q1
 U 1 1 5370319E
 P 4750 2250
@@
 Text Label 3800 2250 0    40   ~ 0
 GATE
-Text Label 4850 2850 1    40   ~ 0
+Text Label 4850 2950 1    40   ~ 0
 SOURCE
 Text Notes 5250 1100 0    40   ~ 0
@@
 Wire Wire Line
 	3000 2450 3000 2550
+Wire Wire Line
+	4900 2250 5000 2250
+Wire Wire Line
+	5000 2250 5000 2650
+Wire Wire Line
+	5000 2650 4850 2650
+Connection ~ 4850 2650
 $EndSCHEMATC
